Commit message: Created seperate srdf files

File: ar3_description/urdf/ar3.urdf.xacro (robot description, xacro)
@@ -5,4 +5,11 @@
 <!-- =================================================================================== -->
 <robot name="ar3">
+  <link name="world" />
+  <link name="world_base"/>
+  <joint name="joint_world_base" type="fixed">
+    <parent link="world"/>
+    <child link="world_base"/>
+    <origin xyz="0 0 0" rpy="0 0 0"/>
+  </joint>
   <link name="base_link">
     <inertial>
@@ -27,4 +34,9 @@
     </collision>
   </link>
+  <joint name="joint_world" type="fixed">
+    <parent link="world_base"/>
+    <child link="base_link"/>
+    <origin xyz="0 0 0" rpy="0 0 0"/>
+  </joint>
   <link name="link_1">
     <inertial>

Commit message: Launches respective srdf for simulated and hardware

File: ar3_description/urdf/ar3.urdf.xacro (robot description, xacro)
@@ -5,4 +5,11 @@
 <!-- =================================================================================== -->
 <robot name="ar3">
+  <link name="world" />
+  <link name="world_base"/>
+  <joint name="joint_world_base" type="fixed">
+    <parent link="world"/>
+    <child link="world_base"/>
+    <origin xyz="0 0 0" rpy="0 0 0"/>
+  </joint>
   <link name="base_link">
     <inertial>

File: ar3_description/urdf/ar3_gazebo.urdf.xacro (robot description, xacro)
@@ -214,23 +214,64 @@
     <limit lower="-2.5848326" upper="2.5848326" effort="100" velocity="100"/>
   </joint>
-  <link name="actuator_1">
-    <inertial>
-      <origin rpy="0 0 0" xyz="0.02 0 0.04"/>
+  <link name="palm">
+    <inertial>
+      <origin rpy="0 0 0" xyz="0 0 0.02"/>
       <mass value="0.013863"/>
       <inertia ixx="1.3596E-06" ixy="3.0585E-13" ixz="5.7102E-14" iyy="1.7157E-06" iyz="6.3369E-09" izz="2.4332E-06"/>
     </inertial>
     <visual>
-      <origin rpy="0 0 0" xyz="0.02 0 0.04"/>
-      <geometry>
-        <box size="0.005 0.04 0.04"/>
-      </geometry>
-      <material name="">
-        <color rgba="1 1 0 1"/>
-      </material>
-    </visual>
-    <collision>
-      <origin rpy="0 0 0" xyz="0.02 0 0.04"/>
-      <geometry>
-        <box size="0.005 0.04 0.04"/>
+      <origin rpy="0 0 0" xyz="0 0 0.02"/>
+      <geometry>
+        <box size="0.1 0.04 0.005"/>
+      </geometry>
+      <material name="">
+        <color rgba="1 1 0 1"/>
+      </material>
+    </visual>
+    <collision>
+      <origin rpy="0 0 0" xyz="0 0 0.02"/>
+      <geometry>
+        <box size="0.1 0.04 0.004"/>
+      </geometry>
+    </collision>
+  </link>
+  <joint name="joint_7" type="fixed">
+    <origin rpy="0 0 3.1416" xyz="0 0 0"/>
+    <parent link="link_6"/>
+    <child link="palm"/>
+  </joint>
+  <link name="camera_link">
+    <!--<visual>
+      <origin rpy="0 0 0" xyz="0 0 0.1"/>
+      <geometry>
+        <box size="0.01 0.01 0.01"/>
+      </geometry>
+      <material name="blue">Gazebo/Blue</material>
+    </visual>-->
+  </link>
+  <joint name="camera_joint" type="fixed">
+    <origin rpy="1.5707 -1.5707 0" xyz="0 0 0.01"/>
+    <parent link="palm"/>
+    <child link="camera_link"/>
+  </joint>
+  <link name="actuator_1">
+    <inertial>
+      <origin rpy="0 0 0" xyz="0.02 0 0.05"/>
+      <mass value="0.013863"/>
+      <inertia ixx="1.3596E-06" ixy="3.0585E-13" ixz="5.7102E-14" iyy="1.7157E-06" iyz="6.3369E-09" izz="2.4332E-06"/>
+    </inertial>
+    <visual>
+      <origin rpy="0 0 0" xyz="0.02 0 0.05"/>
+      <geometry>
+        <box size="0.005 0.04 0.05"/>
+      </geometry>
+      <material name="">
+        <color rgba="1 1 0 1"/>
+      </material>
+    </visual>
+    <collision>
+      <origin rpy="0 0 0" xyz="0.02 0 0.05"/>
+      <geometry>
+        <box size="0.005 0.04 0.05"/>
       </geometry>
     </collision>
@@ -238,5 +279,5 @@
   <joint name="actuator_joint_1" type="prismatic">
     <origin rpy="0 0 3.1416" xyz="0 0 0"/>
-    <parent link="link_6"/>
+    <parent link="palm"/>
     <child link="actuator_1"/>
     <axis xyz="1 0 0"/>
@@ -245,21 +286,21 @@
   <link name="actuator_2">
     <inertial>
-      <origin rpy="0 0 0" xyz="-0.02 0 0.04"/>
+      <origin rpy="0 0 0" xyz="-0.02 0 0.05"/>
       <mass value="0.013863"/>
       <inertia ixx="1.3596E-06" ixy="3.0585E-13" ixz="5.7102E-14" iyy="1.7157E-06" iyz="6.3369E-09" izz="2.4332E-06"/>
     </inertial>
     <visual>
-      <origin rpy="0 0 0" xyz="-0.02 0 0.04"/>
-      <geometry>
-        <box size="0.005 0.04 0.04"/>
-      </geometry>
-      <material name="">
-        <color rgba="1 1 0 1"/>
-      </material>
-    </visual>
-    <collision>
-      <origin rpy="0 0 0" xyz="-0.02 0 0.04"/>
-      <geometry>
-        <box size="0.005 0.04 0.04"/>
+      <origin rpy="0 0 0" xyz="-0.02 0 0.05"/>
+      <geometry>
+        <box size="0.005 0.04 0.05"/>
+      </geometry>
+      <material name="">
+        <color rgba="1 1 0 1"/>
+      </material>
+    </visual>
+    <collision>
+      <origin rpy="0 0 0" xyz="-0.02 0 0.05"/>
+      <geometry>
+        <box size="0.005 0.04 0.05"/>
       </geometry>
     </collision>
@@ -267,5 +308,5 @@
   <joint name="actuator_joint_2" type="prismatic">
     <origin rpy="0 0 3.1416" xyz="0 0 0"/>
-    <parent link="link_6"/>
+    <parent link="palm"/>
     <child link="actuator_2"/>
     <axis xyz="1 0 0"/>
@@ -356,17 +397,58 @@
     </plugin>
   </gazebo>
+  <gazebo reference="camera_link">
+    <sensor name="depth_camera" type="depth">
+      <update_rate>20</update_rate>
+      <camera>
+        <horizontal_fov>1.047198</horizontal_fov>
+        <image>
+          <width>640</width>
+          <height>480</height>
+          <format>R8G8B8</format>
+        </image>
+        <clip>
+          <near>0.05</near>
+          <far>3</far>
+        </clip>
+      </camera>
+      <plugin name="depth_camera_plugin" filename="libgazebo_ros_openni_kinect.so">
+        <baseline>0.2</baseline>
+        <alwaysOn>true</alwaysOn>
+        <updateRate>1.0</updateRate>
+        <cameraName>depth_ir</cameraName>
+        <imageTopicName>/camera/color/image_raw</imageTopicName>
+        <cameraInfoTopicName>/camera/color/camera_info</cameraInfoTopicName>
+        <depthImageTopicName>/camera/depth/image_raw</depthImageTopicName>
+        <depthImageInfoTopicName>/camera/depth/camera_info</depthImageInfoTopicName>
+        <pointCloudTopicName>/camera/depth/points</pointCloudTopicName>
+        <frameName>camera_link</frameName>
+        <pointCloudCutoff>0.1</pointCloudCutoff>
+        <pointCloudCutoffMax>1.5</pointCloudCutoffMax>
+        <distortionK1>0.00000001</distortionK1>
+        <distortionK2>0.00000001</distortionK2>
+        <distortionK3>0.00000001</distortionK3>
+        <distortionT1>0.00000001</distortionT1>
+        <distortionT2>0.00000001</distortionT2>
+        <CxPrime>0</CxPrime>
+        <Cx>0</Cx>
+        <Cy>0</Cy>
+        <focalLength>0</focalLength>
+        <hackBaseline>0</hackBaseline>
+      </plugin>
+    </sensor>
+  </gazebo>
   <gazebo>
    <plugin name="gazebo_grasp_fix" filename="libgazebo_grasp_fix.so">
         <arm>
            <arm_name>ar3</arm_name>
-           <palm_link> link_6  </palm_link>
+           <palm_link>link_6</palm_link>
            <gripper_link> actuator_1 </gripper_link>
            <gripper_link> actuator_2 </gripper_link>
         </arm>
        <forces_angle_tolerance>100</forces_angle_tolerance>
-       <update_rate>8</update_rate>
+       <update_rate>10</update_rate>
        <grip_count_threshold>1</grip_count_threshold>
        <max_grip_count>4</max_grip_count>
-       <release_tolerance>0.007</release_tolerance>
+       <release_tolerance>0.009</release_tolerance>
        <disable_collisions_on_attach>false</disable_collisions_on_attach>
        <contact_topic>__default_topic__</contact_topic>
@@ -394,4 +476,7 @@
       <selfCollide>true</selfCollide>
   </gazebo>
+  <gazebo reference="palm">
+    <selfCollide>true</selfCollide>
+  </gazebo>
   <gazebo reference="actuator_1">
       <selfCollide>true</selfCollide>
