Commit message: Added new gripper

File: ar3_description/urdf/ar3_gazebo_.urdf.xacro (robot description, xacro)
@@ -216,22 +216,21 @@
   <link name="palm">
     <inertial>
-      <origin rpy="0 3.1415 0" xyz="-0.025 0 -0.003"/>
+      <origin rpy="0 0 0" xyz="0 0 0.02"/>
       <mass value="0.013863"/>
       <inertia ixx="1.3596E-06" ixy="3.0585E-13" ixz="5.7102E-14" iyy="1.7157E-06" iyz="6.3369E-09" izz="2.4332E-06"/>
     </inertial>
     <visual>
-      <origin rpy="0 3.1415 0" xyz="-0.025 0 -0.003"/>
-      <geometry>
-        <!--<box size="0.1 0.04 0.005"/>-->
-        <mesh filename="package://ar3_description/meshes/gripper_palm.STL" scale="0.01 0.01 0.01"/>
-      </geometry>
-      <material name="">
-        <color rgba="1 1 0 1"/>
-      </material>
-    </visual>
-    <collision>
-      <origin rpy="0 3.1415 0" xyz="-0.025 0 -0.003"/>
-      <geometry>
-        <mesh filename="package://ar3_description/meshes/gripper_palm.STL" scale="0.01 0.01 0.01"/>
+      <origin rpy="0 0 0" xyz="0 0 0.02"/>
+      <geometry>
+        <box size="0.1 0.04 0.005"/>
+      </geometry>
+      <material name="">
+        <color rgba="1 1 0 1"/>
+      </material>
+    </visual>
+    <collision>
+      <origin rpy="0 0 0" xyz="0 0 0.02"/>
+      <geometry>
+        <box size="0.1 0.04 0.004"/>
       </geometry>
     </collision>
@@ -258,92 +257,59 @@
   <link name="actuator_1">
     <inertial>
-    <!-- -0.02 0.02 0 -->
-      <origin rpy="0 3.1415 1.0472" xyz="0 0 0.007"/>
+      <origin rpy="0 0 0" xyz="0.02 0 0.05"/>
       <mass value="0.013863"/>
       <inertia ixx="1.3596E-06" ixy="3.0585E-13" ixz="5.7102E-14" iyy="1.7157E-06" iyz="6.3369E-09" izz="2.4332E-06"/>
     </inertial>
     <visual>
-      <origin rpy="0 3.1415 1.0472" xyz="0 0 0.007"/>
-      <geometry>
-        <mesh filename="package://ar3_description/meshes/gripper_link.STL" scale="0.01 0.01 0.01"/>
-      </geometry>
-      <material name="">
-        <color rgba="1 1 0 1"/>
-      </material>
-    </visual>
-    <collision>
-      <origin rpy="0 3.1415 1.0472" xyz="0 0 0.007"/>
-      <geometry>
-        <mesh filename="package://ar3_description/meshes/gripper_link.STL" scale="0.01 0.01 0.01"/>
-      </geometry>
-    </collision>
-  </link>
-  <joint name="actuator_joint_1" type="revolute">
-    <!--0.0195 -0.0124 0.045  -->
-    <origin rpy="0 0 3.1416" xyz="0.0195 -0.0124 0.043"/>
+      <origin rpy="0 0 0" xyz="0.02 0 0.05"/>
+      <geometry>
+        <box size="0.005 0.04 0.05"/>
+      </geometry>
+      <material name="">
+        <color rgba="1 1 0 1"/>
+      </material>
+    </visual>
+    <collision>
+      <origin rpy="0 0 0" xyz="0.02 0 0.05"/>
+      <geometry>
+        <box size="0.005 0.04 0.05"/>
+      </geometry>
+    </collision>
+  </link>
+  <joint name="actuator_joint_1" type="prismatic">
+    <origin rpy="0 0 3.1416" xyz="0 0 0"/>
     <parent link="palm"/>
     <child link="actuator_1"/>
-    <axis xyz="0.5235 1.0471 0"/>
-    <limit lower="-0.523" upper="0.7854" effort="100" velocity="100"/>
+    <axis xyz="1 0 0"/>
+    <limit lower="-0.04" upper="0.04" effort="20" velocity="20"/>
   </joint>
   <link name="actuator_2">
     <inertial>
-      <origin rpy="0 3.1415 2.094" xyz="0 0 0.007"/>
+      <origin rpy="0 0 0" xyz="-0.02 0 0.05"/>
       <mass value="0.013863"/>
       <inertia ixx="1.3596E-06" ixy="3.0585E-13" ixz="5.7102E-14" iyy="1.7157E-06" iyz="6.3369E-09" izz="2.4332E-06"/>
     </inertial>
     <visual>
-      <origin rpy="0 3.1415 2.094" xyz="0 0 0.007"/>
-      <geometry>
-        <mesh filename="package://ar3_description/meshes/gripper_link.STL" scale="0.01 0.01 0.01"/>
-      </geometry>
-      <material name="">
-        <color rgba="1 1 0 1"/>
-      </material>
-    </visual>
-    <collision>
-      <origin rpy="0 3.1415 2.094" xyz="0 0 0.007"/>
-      <geometry>
-        <mesh filename="package://ar3_description/meshes/gripper_link.STL" scale="0.01 0.01 0.01"/>
-      </geometry>
-    </collision>
-  </link>
-  <joint name="actuator_joint_2" type="revolute">
-  <!-- -0.0195 -0.009 0.045 -->
-    <origin rpy="0 0 0" xyz="-0.0175 -0.009 0.043"/>
+      <origin rpy="0 0 0" xyz="-0.02 0 0.05"/>
+      <geometry>
+        <box size="0.005 0.04 0.05"/>
+      </geometry>
+      <material name="">
+        <color rgba="1 1 0 1"/>
+      </material>
+    </visual>
+    <collision>
+      <origin rpy="0 0 0" xyz="-0.02 0 0.05"/>
+      <geometry>
+        <box size="0.005 0.04 0.05"/>
+      </geometry>
+    </collision>
+  </link>
+  <joint name="actuator_joint_2" type="prismatic">
+    <origin rpy="0 0 3.1416" xyz="0 0 0"/>
     <parent link="palm"/>
     <child link="actuator_2"/>
-    <axis xyz="-0.5235 1.0471 0"/>
-    <limit lower="-0.523" upper="0.7854" effort="100" velocity="100"/>
-  </joint>
-  <link name="actuator_3">
-    <inertial>
-      <origin rpy="0 3.1415 0" xyz="0 -0.001 0.007"/>
-      <mass value="0.013863"/>
-      <inertia ixx="1.3596E-06" ixy="3.0585E-13" ixz="5.7102E-14" iyy="1.7157E-06" iyz="6.3369E-09" izz="2.4332E-06"/>
-    </inertial>
-    <visual>
-      <origin rpy="0 3.1415 0" xyz="0 -0.001 0.007"/>
-      <geometry>
-        <mesh filename="package://ar3_description/meshes/gripper_link.STL" scale="0.01 0.01 0.01"/>
-      </geometry>
-      <material name="">
-        <color rgba="1 1 0 1"/>
-      </material>
-    </visual>
-    <collision>
-      <origin rpy="0 3.1415 0" xyz="0 -0.001 0.007"/>
-      <geometry>
-        <mesh filename="package://ar3_description/meshes/gripper_link.STL" scale="0.01 0.01 0.01"/>
-      </geometry>
-    </collision>
-  </link>
-  <joint name="actuator_joint_3" type="revolute">
-  <!-- 0.001 0.017 0.045 -->
-    <origin rpy="0 0 0" xyz="0.001 0.022 0.043"/>
-    <parent link="palm"/>
-    <child link="actuator_3"/>
     <axis xyz="1 0 0"/>
-    <limit lower="-0.523" upper="0.7854" effort="100" velocity="100"/>
+    <limit lower="-0.04" upper="0.04" effort="20" velocity="20"/>
   </joint>
   <transmission name="transmission_1">
@@ -423,14 +389,4 @@
       </joint>
       <actuator name="motor_8">
-          <hardwareInterface>hardware_interface/PositionJointInterface</hardwareInterface>
-          <mechanicalReduction>1</mechanicalReduction>
-      </actuator>
-  </transmission>
-  <transmission name="transmission_9">
-      <type>transmission_interface/SimpleTransmission</type>
-      <joint name="actuator_joint_3">
-          <hardwareInterface>hardware_interface/PositionJointInterface</hardwareInterface>
-      </joint>
-      <actuator name="motor_9">
           <hardwareInterface>hardware_interface/PositionJointInterface</hardwareInterface>
           <mechanicalReduction>1</mechanicalReduction>
@@ -489,5 +445,4 @@
            <gripper_link> actuator_1 </gripper_link>
            <gripper_link> actuator_2 </gripper_link>
-           <gripper_link> actuator_3 </gripper_link>
         </arm>
        <forces_angle_tolerance>100</forces_angle_tolerance>
@@ -530,6 +485,3 @@
       <selfCollide>true</selfCollide>
   </gazebo>
-    <gazebo reference="actuator_3">
-      <selfCollide>true</selfCollide>
-  </gazebo>
 </robot>
