Commit message: added gripper on one arm

File: ar3_description/urdf/ar3_gazebo.urdf.xacro (robot description, xacro)
@@ -207,4 +207,5 @@
     <limit lower="-2.5848326" upper="2.5848326" effort="100" velocity="100"/>
   </joint>
+  <joint name=""
   <transmission name="transmission_1">
     <type>transmission_interface/SimpleTransmission</type>

File: ar3_description/urdf/left_ar3_gazebo.urdf.xacro (robot description, xacro)
@@ -206,4 +206,62 @@
     <axis xyz="0 0 1"/>
     <limit lower="-2.5848326" upper="2.5848326" effort="100" velocity="100"/>
+  </joint>
+  <link name="actuator_1">
+    <inertial>
+      <origin rpy="0 0 0" xyz="0.02 0 0.04"/>
+      <mass value="0.013863"/>
+      <inertia ixx="1.3596E-06" ixy="3.0585E-13" ixz="5.7102E-14" iyy="1.7157E-06" iyz="6.3369E-09" izz="2.4332E-06"/>
+    </inertial>
+    <visual>
+      <origin rpy="0 0 0" xyz="0.02 0 0.04"/>
+      <geometry>
+        <box size="0.005 0.04 0.04"/>
+      </geometry>
+      <material name="">
+        <color rgba="1 1 0 1"/>
+      </material>
+    </visual>
+    <collision>
+      <origin rpy="0 0 0" xyz="0.02 0 0.04"/>
+      <geometry>
+        <box size="0.005 0.04 0.04"/>
+      </geometry>
+    </collision>
+  </link>
+  <joint name="actuator_joint_1" type="prismatic">
+    <origin rpy="0 0 3.1416" xyz="0 0 0"/>
+    <parent link="link_6"/>
+    <child link="actuator_1"/>
+    <axis xyz="1 0 0"/>
+    <limit lower="-0.04" upper="0.04" effort="20" velocity="20"/>
+  </joint>
+  <link name="actuator_2">
+    <inertial>
+      <origin rpy="0 0 0" xyz="-0.02 0 0.04"/>
+      <mass value="0.013863"/>
+      <inertia ixx="1.3596E-06" ixy="3.0585E-13" ixz="5.7102E-14" iyy="1.7157E-06" iyz="6.3369E-09" izz="2.4332E-06"/>
+    </inertial>
+    <visual>
+      <origin rpy="0 0 0" xyz="-0.02 0 0.04"/>
+      <geometry>
+        <box size="0.005 0.04 0.04"/>
+      </geometry>
+      <material name="">
+        <color rgba="1 1 0 1"/>
+      </material>
+    </visual>
+    <collision>
+      <origin rpy="0 0 0" xyz="-0.02 0 0.04"/>
+      <geometry>
+        <box size="0.005 0.04 0.04"/>
+      </geometry>
+    </collision>
+  </link>
+  <joint name="actuator_joint_2" type="prismatic">
+    <origin rpy="0 0 3.1416" xyz="0 0 0"/>
+    <parent link="link_6"/>
+    <child link="actuator_2"/>
+    <axis xyz="1 0 0"/>
+    <limit lower="-0.04" upper="0.04" effort="20" velocity="20"/>
   </joint>
   <transmission name="transmission_1">
@@ -267,4 +325,24 @@
       </actuator>
   </transmission>
+  <transmission name="transmission_7">
+      <type>transmission_interface/SimpleTransmission</type>
+      <joint name="actuator_joint_1">
+          <hardwareInterface>hardware_interface/PositionJointInterface</hardwareInterface>
+      </joint>
+      <actuator name="motor_7">
+          <hardwareInterface>hardware_interface/PositionJointInterface</hardwareInterface>
+          <mechanicalReduction>1</mechanicalReduction>
+      </actuator>
+  </transmission>
+  <transmission name="transmission_8">
+      <type>transmission_interface/SimpleTransmission</type>
+      <joint name="actuator_joint_2">
+          <hardwareInterface>hardware_interface/PositionJointInterface</hardwareInterface>
+      </joint>
+      <actuator name="motor_8">
+          <hardwareInterface>hardware_interface/PositionJointInterface</hardwareInterface>
+          <mechanicalReduction>1</mechanicalReduction>
+      </actuator>
+  </transmission>
   <gazebo>
     <plugin name="gazebo_ros_control" filename="libgazebo_ros_control.so">
@@ -292,3 +370,9 @@
       <selfCollide>true</selfCollide>
   </gazebo>
+  <gazebo reference="actuator_1">
+      <selfCollide>true</selfCollide>
+  </gazebo>
+  <gazebo reference="actuator_2">
+      <selfCollide>true</selfCollide>
+  </gazebo>
 </robot>

Commit message: both arms have grippers

File: ar3_description/urdf/ar3_gazebo.urdf.xacro (robot description, xacro)
@@ -4,6 +4,13 @@
 <!-- |    EDITING THIS FILE BY HAND IS NOT RECOMMENDED but it was unfortunately        | -->
 <!-- =================================================================================== -->
-<robot name="ar3">
+<robot xmlns:xacro="http://www.ros.org/wiki/xacro" name="ar3">
+  <xacro:arg name="x_pos" default="0"/>
   <link name="world" />
+  <link name="world_base"/>
+  <joint name="joint_world_base" type="fixed">
+    <parent link="world"/>
+    <child link="world_base"/>
+    <origin xyz="$(arg x_pos) 0 0" rpy="0 0 0"/>
+  </joint>
   <link name="base_link">
     <inertial>
@@ -29,5 +36,5 @@
   </link>
   <joint name="joint_world" type="fixed">
-    <parent link="world"/>
+    <parent link="world_base"/>
     <child link="base_link"/>
     <origin xyz="0 0 0" rpy="0 0 0" />
@@ -207,5 +214,62 @@
     <limit lower="-2.5848326" upper="2.5848326" effort="100" velocity="100"/>
   </joint>
-  <joint name=""
+  <link name="actuator_1">
+    <inertial>
+      <origin rpy="0 0 0" xyz="0.02 0 0.04"/>
+      <mass value="0.013863"/>
+      <inertia ixx="1.3596E-06" ixy="3.0585E-13" ixz="5.7102E-14" iyy="1.7157E-06" iyz="6.3369E-09" izz="2.4332E-06"/>
+    </inertial>
+    <visual>
+      <origin rpy="0 0 0" xyz="0.02 0 0.04"/>
+      <geometry>
+        <box size="0.005 0.04 0.04"/>
+      </geometry>
+      <material name="">
+        <color rgba="1 1 0 1"/>
+      </material>
+    </visual>
+    <collision>
+      <origin rpy="0 0 0" xyz="0.02 0 0.04"/>
+      <geometry>
+        <box size="0.005 0.04 0.04"/>
+      </geometry>
+    </collision>
+  </link>
+  <joint name="actuator_joint_1" type="prismatic">
+    <origin rpy="0 0 3.1416" xyz="0 0 0"/>
+    <parent link="link_6"/>
+    <child link="actuator_1"/>
+    <axis xyz="1 0 0"/>
+    <limit lower="-0.04" upper="0.04" effort="20" velocity="20"/>
+  </joint>
+  <link name="actuator_2">
+    <inertial>
+      <origin rpy="0 0 0" xyz="-0.02 0 0.04"/>
+      <mass value="0.013863"/>
+      <inertia ixx="1.3596E-06" ixy="3.0585E-13" ixz="5.7102E-14" iyy="1.7157E-06" iyz="6.3369E-09" izz="2.4332E-06"/>
+    </inertial>
+    <visual>
+      <origin rpy="0 0 0" xyz="-0.02 0 0.04"/>
+      <geometry>
+        <box size="0.005 0.04 0.04"/>
+      </geometry>
+      <material name="">
+        <color rgba="1 1 0 1"/>
+      </material>
+    </visual>
+    <collision>
+      <origin rpy="0 0 0" xyz="-0.02 0 0.04"/>
+      <geometry>
+        <box size="0.005 0.04 0.04"/>
+      </geometry>
+    </collision>
+  </link>
+  <joint name="actuator_joint_2" type="prismatic">
+    <origin rpy="0 0 3.1416" xyz="0 0 0"/>
+    <parent link="link_6"/>
+    <child link="actuator_2"/>
+    <axis xyz="1 0 0"/>
+    <limit lower="-0.04" upper="0.04" effort="20" velocity="20"/>
+  </joint>
   <transmission name="transmission_1">
     <type>transmission_interface/SimpleTransmission</type>
@@ -268,4 +332,24 @@
       </actuator>
   </transmission>
+  <transmission name="transmission_7">
+      <type>transmission_interface/SimpleTransmission</type>
+      <joint name="actuator_joint_1">
+          <hardwareInterface>hardware_interface/PositionJointInterface</hardwareInterface>
+      </joint>
+      <actuator name="motor_7">
+          <hardwareInterface>hardware_interface/PositionJointInterface</hardwareInterface>
+          <mechanicalReduction>1</mechanicalReduction>
+      </actuator>
+  </transmission>
+  <transmission name="transmission_8">
+      <type>transmission_interface/SimpleTransmission</type>
+      <joint name="actuator_joint_2">
+          <hardwareInterface>hardware_interface/PositionJointInterface</hardwareInterface>
+      </joint>
+      <actuator name="motor_8">
+          <hardwareInterface>hardware_interface/PositionJointInterface</hardwareInterface>
+          <mechanicalReduction>1</mechanicalReduction>
+      </actuator>
+  </transmission>
   <gazebo>
     <plugin name="gazebo_ros_control" filename="libgazebo_ros_control.so">
@@ -293,3 +377,9 @@
       <selfCollide>true</selfCollide>
   </gazebo>
+  <gazebo reference="actuator_1">
+      <selfCollide>true</selfCollide>
+  </gazebo>
+  <gazebo reference="actuator_2">
+      <selfCollide>true</selfCollide>
+  </gazebo>
 </robot>

Commit message: Added colliders to prevent gripper/ground collision

File: ar3_description/urdf/ar3_gazebo.urdf.xacro (robot description, xacro)
@@ -6,11 +6,20 @@
 <robot xmlns:xacro="http://www.ros.org/wiki/xacro" name="ar3_arm">
   <xacro:arg name="x_pos" default="0"/>
+  <xacro:arg name="for_moveit" default="true"/>
   <link name="world"/>
-  <link name="world_base"/>
-<joint name="world_joint" type="fixed">
-  <parent link="world"/>
-  <child link="world_base"/>
-  <origin xyz="0 0 0" rpy="0 0 0"/>
-</joint>
+  <!-- Thin Box below arm provides collision on ground -->
+  <link name="world_base">
+    <collision>
+      <origin rpy="0 0 0" xyz="0 0 0.001"/>
+      <geometry>
+        <box size="2 2 0.0001"/>
+      </geometry>
+    </collision>
+  </link>
+  <joint name="world_joint" type="fixed">
+    <parent link="world"/>
+    <child link="world_base"/>
+    <origin xyz="0 0 0" rpy="0 0 0"/>
+  </joint>
   <link name="base_link">
     <inertial>
@@ -213,4 +222,20 @@
     <axis xyz="0 0 1"/>
     <limit lower="-2.5848326" upper="2.5848326" effort="100" velocity="100"/>
+  </joint>
+  <!-- Box that provides gripper collider only for moveit so gazebo does not simulate collisions -->
+  <link name="gripper_collider">
+    <xacro:if value="$(arg for_moveit)">
+      <collision>
+        <origin rpy="0 0 0" xyz="0 0 0.05"/>
+        <geometry>
+          <box size="0.1 0.1 0.05"/>
+        </geometry>
+      </collision>
+    </xacro:if>
+  </link>
+  <joint name="grip_collide_joint" type="fixed">
+    <origin rpy="0 0 0" xyz="0 0 0"/>
+    <parent link="link_6"/>
+    <child link="gripper_collider"/>
   </joint>
   <link name="camera_link">

Commit message: Found patch to terrible srdf loading issue

File: ar3_description/urdf/ar3_gazebo.urdf.xacro (robot description, xacro)
@@ -4,5 +4,5 @@
 <!-- |    EDITING THIS FILE BY HAND IS NOT RECOMMENDED but it was unfortunately        | -->
 <!-- =================================================================================== -->
-<robot xmlns:xacro="http://www.ros.org/wiki/xacro" name="ar3_arm">
+<robot xmlns:xacro="http://www.ros.org/wiki/xacro" name="ar3">
   <xacro:arg name="x_pos" default="0"/>
   <xacro:arg name="for_moveit" default="true"/>

File: ar3_moveit_config/config/ar3_old.srdf.xacro (robot description, xacro)
@@ -1,8 +1,5 @@
 <?xml version="1.0" ?>
-<!--This does not replace URDF, and is not an extension of URDF.
-    This is a format for representing semantic information about the robot structure.
-    A URDF file must exist for this robot as well, where the joints and the links that are referenced are defined
--->
-<robot name="ar3">
+<!-- Note: This should be the only srdf needed for the ar3, I will be deleting the ar3_hardware and ar3_gripper_gazebo once I know they are no longer needed.-->
+<robot name="ar3_arm">
     <!--GROUPS: Representation of a set of joints and links. This can be useful for specifying DOF to plan for, defining arms, end effectors, etc-->
     <!--LINKS: When a link is specified, the parent joint of that link (if it exists) is automatically included-->
@@ -16,5 +13,5 @@
         <joint name="joint_4" />
         <joint name="joint_5" />
-        <joint name="joint_6"/>
+        <joint name="joint_6" />
     </group>
     <!--GROUP STATES: Purpose: Define a named state for a particular group, in terms of joint values. This is useful to define states like 'folded arms'-->
@@ -36,8 +33,6 @@
     </group_state>
     <!--END EFFECTOR: Purpose: Represent information about an end effector.-->
-    <end_effector name="gripper" parent_link="link_6" group="manipulator" />
-    <virtual_joint name="world_joint" type="fixed" parent_frame="world" child_link="base_link"/>
+    <end_effector name="end_effector" parent_link="link_6" group="manipulator" />
     <!--DISABLE COLLISIONS: By default it is assumed that any link of the robot could potentially come into collision with any other link in the robot. This tag disables collision checking between a specified pair of links. -->
-    <disable_collisions link1="world_base" link2="base_link" reason="Adjacent"/>
     <disable_collisions link1="base_link" link2="link_1" reason="Adjacent" />
     <disable_collisions link1="link_1" link2="link_2" reason="Adjacent" />
@@ -49,6 +44,3 @@
     <disable_collisions link1="link_4" link2="link_5" reason="Adjacent" />
     <disable_collisions link1="link_5" link2="link_6" reason="Adjacent" />
-    <disable_collisions link1="link_6" link2="gripper_collider" reason="Adjacent"/>
-    <disable_collisions link1="link_5" link2="gripper_collider" reason="Adjacent"/>
-    <disable_collisions link1="link_4" link2="gripper_collider" reason="Adjacent"/>
 </robot>
